File: PCB/main/microcontroller_interfacing.kicad_sch (KiCad schematic)
At the start: 0 parts

Commit message: added digital sensors
Other:
- company: (none) -> University of Cape Town
- title: (none) -> DiscoverAir HAT
Changed lines of the file:
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@@
 (kicad_sch (version 20211123) (generator eeschema)
   (paper "A4")
+  (title_block
+    (title "DiscoverAir HAT")
+    (rev "V0.0")
+    (company "University of Cape Town")
+    (comment 4 "@Authors: Justin Pead, Mark Njoroge")
+  )
   (text "Memory Element and which pins you wish to use.\ndebugging capabilities to test it\n"
     (at 129.54 89.535 0)
